File: interfaces.kicad_sch (KiCad schematic)
At the start: 25 parts, among them J2 Pico 3PIN SWD, J3 Pico 3PIN UART, J4 BATT, Q2 2N7002, Q3 2N7002, SW1 BOOT, SW2 RESET, SW3 RotaryEncoder_Switch, SW4 SW_SPST, U8 4011

Commit message: feat: optimizations
Parts:
- added J8: TALLYLIGHT, Connector_JST:JST_PH_S3B-PH-SM4-TB_1x03-1MP_P2.00mm_Horizontal, symbol Connector_Generic_MountingPin:Conn_01x03_MountingPin
Connections:
- net GND: now also J8.3 (Pin_3), J8.MP (MountPin)
- new net +VIN: J8.1 (Pin_1)
- new net TALLY_OUT: J8.2 (Pin_2)
