File: mcu.kicad_sch (KiCad schematic)
At the start: 14 parts, among them U1 RP2040

Commit message: feat: optimizations
Connections:
- net GPIO12: now reaches U1.15 (GPIO12)
- no-connect marks 8 -> 7
Changed lines of the file:
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@@
-	)
-	(no_connect
-		(at 124.46 90.17)
 	)
 	(no_connect
@@
 		)
 	)
+	(hierarchical_label "GPIO12"
+		(shape input)
+		(at 124.46 90.17 0)
+		(fields_autoplaced yes)
+		(effects
+			(font
+				(size 1.27 1.27)
+				(bold yes)
+			)
+			(justify left)
+		)
+	)
