File: power.kicad_sch (KiCad schematic)
At the start: 15 parts, among them Q1 AO3401A, U2 TP4056X, U3 AMS1117-3.3

Commit message: feat: optimizations
Connections:
- net LDO_VIN renamed +VIN
Changed lines of the file:
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@@
 	)
 	(junction
+		(at 138.43 54.61)
+		(diameter 0)
+		(color 0 0 0 0)
+	)
+	(junction
 		(at 160.02 67.31)
 		(diameter 0)
@@
 	(wire
 		(pts
-			(xy 129.54 54.61) (xy 148.59 54.61)
+			(xy 129.54 54.61) (xy 138.43 54.61)
 		)
 		(stroke
@@
 	(wire
 		(pts
+			(xy 138.43 45.72) (xy 138.43 54.61)
+		)
+		(stroke
+			(width 0)
+			(type default)
+		)
+	)
+	(wire
+		(pts
 			(xy 72.39 35.56) (xy 87.63 35.56)
 		)
@@
 	(wire
 		(pts
+			(xy 138.43 54.61) (xy 148.59 54.61)
+		)
+		(stroke
+			(width 0)
+			(type default)
+		)
+	)
+	(wire
+		(pts
 			(xy 99.06 48.26) (xy 99.06 54.61)
 		)
@@
 		)
 	)
-	(label "LDO_VIN"
-		(at 140.97 54.61 0)
-		(fields_autoplaced yes)
-		(effects
-			(font
-				(size 1.27 1.27)
-			)
-			(justify left bottom)
-		)
-	)
 	(label "CHRG_STAT_1"
 		(at 72.39 40.64 0)
@@
 					(unit 1)
 				)
+			)
+		)
+	)
+	(symbol
+		(lib_id "power:+3V3")
+		(at 138.43 45.72 0)
+		(unit 1)
+		(exclude_from_sim no)
+		(in_bom yes)
+		(on_board yes)
+		(dnp no)
+		(fields_autoplaced yes)
+		(property "Reference" "#PWR058"
+			(at 138.43 49.53 0)
+			(effects
+				(font
+					(size 1.27 1.27)
+				)
+				(hide yes)
+			)
+		)
+		(property "Value" "+VIN"
+			(at 138.43 40.64 0)
+			(effects
+				(font
+					(size 1.27 1.27)
+				)
+			)
+		)
+		(property "Footprint" ""
+			(at 138.43 45.72 0)
+			(effects
+				(font
+					(size 1.27 1.27)
+				)
+				(hide yes)
+			)
+		)
+		(property "Datasheet" ""
+			(at 138.43 45.72 0)
+			(effects
+				(font
+					(size 1.27 1.27)
+				)
+				(hide yes)
+			)
+		)
+		(property "Description" "Power symbol creates a global label with name \"+VIN\""
+			(at 138.43 45.72 0)
+			(effects
+				(font
+					(size 1.27 1.27)
+				)
+				(hide yes)
+			)
+		)
+		(pin "1"
+		)
+		(instances
+			(project "tallytime"
+				(path "/7e984edf-b9a3-46d5-a368-ca341108e5fe/a274986d-3ac0-473e-9272-3b44489a97fa"
+					(reference "#PWR058")
+					(unit 1)
+				)
