File: tallytime.kicad_sch (KiCad schematic)
At the start: 2 parts

Commit message: feat: optimizations
Other:
- sheet Interfaces ports: added TALLY_OUT; removed none
- sheet MCU ports: added GPIO12; removed none
Changed lines of the file:
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@@
+	(wire
+		(pts
+			(xy 165.1 116.84) (xy 177.8 116.84)
+		)
+		(stroke
+			(width 0)
+			(type default)
+		)
+	)
 	(wire
 		(pts
@@
 	(wire
 		(pts
-			(xy 165.1 118.11) (xy 177.8 118.11)
+			(xy 165.1 120.65) (xy 177.8 120.65)
 		)
 		(stroke
@@
 	(wire
 		(pts
+			(xy 165.1 125.73) (xy 177.8 125.73)
+		)
+		(stroke
+			(width 0)
+			(type default)
+		)
+	)
+	(bus
+		(pts
+			(xy 111.76 58.42) (xy 111.76 64.77)
+		)
+		(stroke
+			(width 0)
+			(type default)
+		)
+	)
+	(bus
+		(pts
+			(xy 132.08 137.16) (xy 134.62 137.16)
+		)
+		(stroke
+			(width 0)
+			(type default)
+		)
+	)
+	(bus
+		(pts
+			(xy 165.1 72.39) (xy 168.91 72.39)
+		)
+		(stroke
+			(width 0)
+			(type default)
+		)
+	)
+	(bus
+		(pts
+			(xy 134.62 137.16) (xy 137.16 137.16)
+		)
+		(stroke
+			(width 0)
+			(type default)
+		)
+	)
+	(wire
+		(pts
+			(xy 165.1 129.54) (xy 177.8 129.54)
+		)
+		(stroke
+			(width 0)
+			(type default)
+		)
+	)
+	(wire
+		(pts
+			(xy 101.6 87.63) (xy 114.3 87.63)
+		)
+		(stroke
+			(width 0)
+			(type default)
+		)
+	)
+	(wire
+		(pts
+			(xy 175.26 102.87) (xy 177.8 102.87)
+		)
+		(stroke
+			(width 0)
+			(type default)
+		)
+	)
+	(bus
+		(pts
+			(xy 137.16 137.16) (xy 139.7 137.16)
+		)
+		(stroke
+			(width 0)
+			(type default)
+		)
+	)
+	(wire
+		(pts
+			(xy 142.24 132.08) (xy 142.24 146.05)
+		)
+		(stroke
+			(width 0)
+			(type default)
+		)
+	)
+	(wire
+		(pts
+			(xy 147.32 132.08) (xy 147.32 146.05)
+		)
+		(stroke
+			(width 0)
+			(type default)
+		)
+	)
+	(wire
+		(pts
+			(xy 101.6 77.47) (xy 114.3 77.47)
+		)
+		(stroke
+			(width 0)
+			(type default)
+		)
+	)
+	(wire
+		(pts
+			(xy 101.6 80.01) (xy 114.3 80.01)
+		)
+		(stroke
+			(width 0)
+			(type default)
+		)
+	)
+	(wire
+		(pts
 			(xy 165.1 123.19) (xy 177.8 123.19)
-		)
-		(stroke
-			(width 0)
-			(type default)
-		)
-	)
-	(bus
-		(pts
-			(xy 111.76 58.42) (xy 111.76 64.77)
-		)
-		(stroke
-			(width 0)
-			(type default)
-		)
-	)
-	(bus
-		(pts
-			(xy 132.08 137.16) (xy 134.62 137.16)
-		)
-		(stroke
-			(width 0)
-			(type default)
-		)
-	)
-	(bus
-		(pts
-			(xy 165.1 72.39) (xy 168.91 72.39)
-		)
-		(stroke
-			(width 0)
-			(type default)
-		)
-	)
-	(bus
-		(pts
-			(xy 134.62 137.16) (xy 137.16 137.16)
-		)
-		(stroke
-			(width 0)
-			(type default)
-		)
-	)
-	(wire
-		(pts
-			(xy 165.1 127) (xy 177.8 127)
-		)
-		(stroke
-			(width 0)
-			(type default)
-		)
-	)
-	(wire
-		(pts
-			(xy 101.6 87.63) (xy 114.3 87.63)
-		)
-		(stroke
-			(width 0)
-			(type default)
-		)
-	)
-	(wire
-		(pts
-			(xy 175.26 102.87) (xy 177.8 102.87)
-		)
-		(stroke
-			(width 0)
-			(type default)
-		)
-	)
-	(bus
-		(pts
-			(xy 137.16 137.16) (xy 139.7 137.16)
-		)
-		(stroke
-			(width 0)
-			(type default)
-		)
-	)
-	(wire
-		(pts
-			(xy 142.24 132.08) (xy 142.24 146.05)
-		)
-		(stroke
-			(width 0)
-			(type default)
-		)
-	)
-	(wire
-		(pts
-			(xy 147.32 132.08) (xy 147.32 146.05)
-		)
-		(stroke
-			(width 0)
-			(type default)
-		)
-	)
-	(wire
-		(pts
-			(xy 101.6 77.47) (xy 114.3 77.47)
-		)
-		(stroke
-			(width 0)
-			(type default)
-		)
-	)
-	(wire
-		(pts
-			(xy 101.6 80.01) (xy 114.3 80.01)
-		)
-		(stroke
-			(width 0)
-			(type default)
-		)
-	)
-	(wire
-		(pts
-			(xy 165.1 120.65) (xy 177.8 120.65)
 		)
 		(stroke
@@
 		)
 		(pin "GPIO23" input
+			(at 165.1 123.19 0)
+			(effects
+				(font
+					(size 1.27 1.27)
+				)
+				(justify right)
+			)
+		)
+		(pin "GPIO22" input
 			(at 165.1 120.65 0)
 			(effects
@@
 			)
 		)
-		(pin "GPIO22" input
-			(at 165.1 118.11 0)
-			(effects
-				(font
-					(size 1.27 1.27)
-				)
-				(justify right)
-			)
-		)
 		(pin "GPIO24" input
-			(at 165.1 123.19 0)
+			(at 165.1 125.73 0)
 			(effects
 				(font
@@
 		)
 		(pin "GPIO6" input
-			(at 165.1 127 0)
+			(at 165.1 129.54 0)
+			(effects
+				(font
+					(size 1.27 1.27)
+				)
+				(justify right)
+			)
+		)
+		(pin "GPIO12" output
+			(at 165.1 116.84 0)
 			(effects
 				(font
@@
 		)
 		(pin "ENC_B" output
+			(at 177.8 123.19 180)
+			(effects
+				(font
+					(size 1.27 1.27)
+				)
+				(justify left)
+			)
+		)
+		(pin "SW_BACK" output
+			(at 177.8 129.54 180)
+			(effects
+				(font
+					(size 1.27 1.27)
+				)
+				(justify left)
+			)
+		)
+		(pin "ENC_SW" output
+			(at 177.8 125.73 180)
+			(effects
+				(font
+					(size 1.27 1.27)
+				)
+				(justify left)
+			)
+		)
+		(pin "ENC_A" output
 			(at 177.8 120.65 180)
 			(effects
@@
 			)
 		)
-		(pin "SW_BACK" output
-			(at 177.8 127 180)
-			(effects
-				(font
-					(size 1.27 1.27)
-				)
-				(justify left)
-			)
-		)
-		(pin "ENC_SW" output
-			(at 177.8 123.19 180)
-			(effects
-				(font
-					(size 1.27 1.27)
-				)
-				(justify left)
-			)
-		)
-		(pin "ENC_A" output
-			(at 177.8 118.11 180)
-			(effects
-				(font
+		(pin "TALLY_OUT" input
+			(at 177.8 116.84 180)
+			(effects
+				(font

Commit message: v0.1.0
Parts:
- removed JP1: UART_RX, Jumper:SolderJumper-2_P1.3mm_Bridged_Pad1.0x1.5mm, symbol Jumper:SolderJumper_2_Bridged
- removed JP2: UART_TX, Jumper:SolderJumper-2_P1.3mm_Bridged_Pad1.0x1.5mm, symbol Jumper:SolderJumper_2_Bridged
Other:
- removed sheet Interfaces
- removed sheet TimecodeIO
- added sheet Debug (sheets/debug.kicad_sch)
- added sheet Timecode (sheets/timecode.kicad_sch)
- added sheet USB (sheets/usb.kicad_sch)
- sheet Display: file display.kicad_sch -> sheets/display.kicad_sch
- sheet Display ports: added D/C, RES, SCL_MOSI, SDA_SCLK; removed CLK, DC, MOSI, ~{RESET}
- sheet MCU: file mcu.kicad_sch -> sheets/mcu.kicad_sch
- sheet MCU ports: added GPIO0, GPIO1, GPIO10, GPIO11, GPIO13, GPIO14, GPIO15, GPIO16, GPIO17, GPIO18, GPIO19, GPIO2, GPIO25, GPIO26_ADC0, GPIO27_ADC1, GPIO28_ADC2, GPIO29_ADC3, GPIO3, GPIO4, GPIO5, GPIO9, USB_D+, USB_D-; removed DET_IN, DET_OUT, LTC_RX, LTC_TX, SPI0_CS1, SPI0{SCK MOSI MISO}, SPI1_CS1, SPI1_CS2, SPI1{SCK MOSI}, UART0_RX, UART0_TX
- sheet Mechanical: file mechanical.kicad_sch -> sheets/mechanical.kicad_sch
- sheet Power: file power.kicad_sch -> sheets/power.kicad_sch
- sheet Radio: file radio.kicad_sch -> sheets/radio.kicad_sch
- sheet Radio ports: added DIO1, DIO2, DIO3, DIO4, DIO5; removed none
- note removed: "RP2-B2"
- note removed: "Ra-02"
